Commit message: STL Models added !

File: DuckSimROS2/src/biped_descriptions/xacro/cassie_real.xacro (robot description, xacro)
@@ -36,13 +36,13 @@
     </link>
       <gazebo reference="vectorNav">
-    <kp>100000000.0</kp>
-    <kd>10.0</kd>
-    <mu1>0.1</mu1>
-    <mu2>0.1</mu2>
-    <fdir1>1 0 0</fdir1>
-    <maxVel>10.0</maxVel>
-    <minDepth>0.0005</minDepth>
-    <material>Gazebo/Green</material>
-  </gazebo>
+        <kp>100000000.0</kp>
+        <kd>10.0</kd>
+        <mu1>0.1</mu1>
+        <mu2>0.1</mu2>
+        <fdir1>1 0 0</fdir1>
+        <maxVel>10.0</maxVel>
+        <minDepth>0.0005</minDepth>
+        <material>Gazebo/Green</material>
+      </gazebo>
   </xacro:macro>
   <xacro:macro name="pelvis" params="cname color">
@@ -445,8 +445,8 @@
       </hardware>
       <joint name="hip_abduction_${side}">
-        <command_intreface name="effort">
+        <command_interface name="effort">
           <param name="min">-10</param>
           <param name="max">+10</param>
-        </command_intreface>
+        </command_interface>
         <state_interface name="position">
           <param name="initial_value">1.0</param>

Commit message: Tested all joints and DOF of biped duck robot model - RViz2

File: DuckSimROS2/src/biped_descriptions/xacro/cassie_real.xacro (robot description, xacro)
@@ -388,5 +388,5 @@
       <parent link="${side}_pelvis_rotation" />
       <child link="${side}_hip" />
-      <limit lower="0.0" upper="0.0" effort="2000.0" velocity="12.1475" />
+      <limit lower="-0.0" upper="0.0" effort="1.0" velocity="1.0" />
     </joint>
   </xacro:macro>
@@ -432,13 +432,13 @@
     <joint name="toe_joint_${side}" type="revolute">
       <origin xyz="0.408 -0.04 0" rpy="0 0 -1.5"/>
-      <axis xyz="0 0 1"/>
+      <axis xyz="0 1 0"/>
       <parent link="${side}_tarsus" />
       <child link="${side}_toe" />
-      <limit lower="0" upper="0" effort="2000.0" velocity="11.5192" />
+      <limit lower="0" upper="0" effort="0.01" velocity="0.1" />
     </joint>
   </xacro:macro>
   <!-- Transmission Definitions -->
-  <xacro:macro name="hip_rotation_trans" params="side">
-    <ros2_control name="hip_rotation_trans_${side}" type="system">
+  <!-- <xacro:macro name="hip_abduction_trans" params="side">
+    <ros2_control name="hip_abduction_trans_${side}" type="system">
       <hardware>
         <plugin>gazebo_ros2_control/GazeboSystem</plugin>
@@ -457,5 +457,42 @@
     </ros2_control>
   </xacro:macro>
-  <!-- <xacro:macro name="hip_abduction_trans" params="side">
+  <xacro:macro name="hip_rotation_trans" params="side">
+    <ros2_control name="hip_rotation_trans_${side}" type="system">
+      <hardware>
+        <plugin>gazebo_ros2_control/GazeboSystem</plugin>
+      </hardware>
+      <joint name="hip_rotation_${side}">
+        <command_interface name="effort">
+          <param name="min">-10</param>
+          <param name="max">+10</param>
+        </command_interface>
+        <state_interface name="position">
+          <param name="initial_value">1.0</param>
+        </state_interface>
+        <state_interface name="velocity"/>
+        <state_interface name="effort"/>
+      </joint>
+    </ros2_control>
+  </xacro:macro>
+  <xacro:macro name="toe_joint_trans" params="side">
+    <ros2_control name="knee_joint_trans_${side}" type="system">
+      <hardware>
+        <plugin>gazebo_ros2_control/GazeboSystem</plugin>
+      </hardware>
+      <joint name="toe_joint_${side}">
+        <command_interface name="effort">
+          <param name="min">-10</param>
+          <param name="max">+10</param>
+        </command_interface>
+        <state_interface name="position">
+          <param name="initial_value">1.0</param>
+        </state_interface>
+        <state_interface name="velocity"/>
+        <state_interface name="effort"/>
+      </joint>
+    </ros2_control>
+  </xacro:macro> -->
+<!-- ******************************************************************************   -->
+  <xacro:macro name="hip_abduction_trans" params="side">
         <transmission name="hip_abduction_trans_${side}">
         <type>transmission_interface/SimpleTransmission</type>
@@ -468,6 +505,6 @@
         </actuator>
     </transmission>
-  </xacro:macro> -->
-  <!-- <xacro:macro name="hip_rotation_trans" params="side">
+  </xacro:macro>
+  <xacro:macro name="hip_rotation_trans" params="side">
     <transmission name="hip_rotation_trans_${side}">
       <type>transmission_interface/SimpleTransmission</type>
@@ -516,5 +553,5 @@
       </actuator>
     </transmission>
-  </xacro:macro>  -->
+  </xacro:macro>
   <!-- Links -->
   <xacro:vectorNav />
@@ -557,8 +594,7 @@
   <xacro:hip_rotation_trans side="left"/>
   <xacro:hip_rotation_trans side="right"/>
-  <gazebo>
-        <plugin name="gazebo_ros2_control" filename="libgazebo_ros2_control.so">
-          <parameters>$(find biped_descriptions)/config/cassie_efforts.yaml</parameters>
-        </plugin>
-  </gazebo>
+  <xacro:hip_abduction_trans side="left"/>
+  <xacro:hip_abduction_trans side="right"/>
+  <xacro:toe_joint_trans side="left"/>
+  <xacro:toe_joint_trans side="right"/>
 </robot>
